File: KiCad/Updifier/Updifier.kicad_pcb (KiCad board)
At the start: 2 copper layers, 56.5 x 21.6 mm, 36 parts, among them J2 UPDI-IN, J3 UPDI_IN6, J4 HVUPDI_OUT6, J5 HVUPDI-OUT, SW1 SN74LVC1G3157DBVR, SW2 ISL43210IHZ-T, SW3 PTS810SJG250SMTRLFS, U1 ATtiny202-SS, U2 NCP1406SNT1G, U3 MIC2091-1YM5-TR

Commit message: WIP
Parts:
- removed J2: UPDI-IN, Connector_PinHeader_2.54mm:PinHeader_1x03_P2.54mm_Horizontal
- removed J4: HVUPDI_OUT6, Connector_PinHeader_2.54mm:PinHeader_2x03_P2.54mm_Vertical
- C1, C2, C3, C4, C5, C6, C7, C8: footprint Capacitor_SMD:C_0603_1608Metric -> Capacitors_SMD:C_0603
- D2: footprint Diode_SMD:D_SOD-323F -> Diodes_SMD:D_SOD-323F
- F1: footprint Fuse:Fuse_0603_1608Metric -> Resistors_SMD:R_0603
- HV1, VTG1: footprint LED_SMD:LED_0603_1608Metric -> LEDs:LED_0805
- J3: footprint Connector_PinHeader_2.54mm:PinHeader_2x03_P2.54mm_Vertical -> Pin_Headers:Pin_Header_Angled_2x05_Pitch1.00mm
- J5: footprint Connector_PinSocket_2.54mm:PinSocket_1x03_P2.54mm_Horizontal -> 78208-103HLF:78208-103HLF
- L1: footprint Inductor_SMD:L_1008_2520Metric -> L_1008_2520Metric:L_1008_2520Metric
- R10, R11, R12, R3, R4, R5, R6, R8, R9: footprint Resistor_SMD:R_0603_1608Metric -> Resistors_SMD:R_0603
- SW1, SW2: footprint 0_mouser:SOT95P280X145-6N -> TO_SOT_Packages_SMD:SOT-23-6
- SW3: value PTS810SJG250SMTRLFS -> RE-UPDIFY; footprint 0_mouser:PTS810SJG250SMTRLFS -> Buttons_Switches_SMD:SW_SPST_EVPBF
- U1: footprint Package_SO:SOIC-8_3.9x4.9mm_P1.27mm -> Housings_SOIC:SOIC-8_3.9x4.9mm_Pitch1.27mm
- U2: footprint 0_mouser:SOT95P275X110-5N -> TO_SOT_Packages_SMD:SOT-23-5
- U3: footprint 0_mouser:SOT95P280X130-5N -> TO_SOT_Packages_SMD:SOT-23-5
- moved R10 70.7 mm to (108.7, 32.4)
- moved R12 65.3 mm to (107.9, 37.3)
- moved J3 64.7 mm to (93.3, 55.9)
- moved U1 53.1 mm to (102.7, 29.4), turned to 0 degrees
- moved R4 52.3 mm to (108.7, 27.4)
- moved R5 51.4 mm to (93.7, 35.8), turned to 0 degrees
- moved J5 48.9 mm to (123.2, 54.0), turned to 270 degrees
- moved R6 48.7 mm to (90.2, 38.2), turned to 0 degrees
- moved L1 46.5 mm to (83.8, 21.0)
- moved F1 45.6 mm to (76.6, 35.9), turned to 0 degrees
- moved R9 45.5 mm to (108.7, 29.9)
- moved R3 42.1 mm to (90.2, 35.8)
- moved C6 36.3 mm to (78.4, 28.8), turned to 0 degrees
- moved SW2 33.9 mm to (70.2, 30.0)
- moved FID1 32.4 mm to (49.5, 48.9)
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Connections:
- J3 pad 4: (no net) -> Net-(J3-Pad4)
- J3 pad 5: (no net) -> Net-(J3-Pad5)
- SW3 pad 1: /UPDI-SENSE -> GND
- U3 pad 4: (no net) -> Net-(U3-Pad4)
Routing:
- net VTG: track 89.9 -> 0.00 mm, vias 2 -> 0
- net /HV-EN: track 83.9 -> 0.00 mm, vias 2 -> 0
- net VF: track 60.1 -> 0.00 mm, vias 2 -> 0
- net GND: track 58.7 -> 0.00 mm, vias 8 -> 0
- net /HVUPDI-TARGET: track 53.3 -> 0.00 mm
- net /UPDI-EN: track 47.2 -> 0.00 mm, vias 2 -> 0
- net /UPDI-HOST: track 43.1 -> 0.00 mm
- net VTG-PC: track 40.9 -> 0.00 mm
- net /PROG: track 36.1 -> 0.00 mm, vias 1 -> 0
- net /12V: track 34.7 -> 0.00 mm, vias 2 -> 0
- net /UPDI-SENSE: track 31.3 -> 0.00 mm
- net Net-(R12-Pad2): track 12.0 -> 0.00 mm
- net Net-(C4-Pad2): track 11.8 -> 0.00 mm
- net /PWR-SW-EN: track 11.3 -> 0.00 mm
- net /UPDI-KEY: track 10.2 -> 0.00 mm
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- removed copper zone on B.Cu, net GND
Other:
- board outline removed
- board text removed: "4E564D50726F6720"
- board text removed: "DAT"
- board text removed: "GND"
- board text removed: "HV"
- board text removed: "HV-UPDI-TARGET"
- board text removed: "HVUPDI"
- board text removed: "PROG"
- board text removed: "RE-UPDIFY"
- board text removed: "UPDI"
- board text removed: "UPDI-HOST"
- board text removed: "Updi-Key"
- board text removed: "VTG"
- board text removed: "VTG-PC"
- board text removed: "github.com/Dlloydev/UpdiKey"
- board text removed: "v1.0"

Commit message: WIP
Parts:
- removed HV1: ORANGE, LEDs:LED_0805
- removed J3: UPDI_IN6, Pin_Headers:Pin_Header_Angled_2x05_Pitch1.00mm
- removed J5: HVUPDI-OUT, 78208-103HLF:78208-103HLF
- removed R10: 10K, Resistors_SMD:R_0603
- removed R11, R12: 180Ω, Resistors_SMD:R_0603
- removed SW2: ISL43210IHZ-T, TO_SOT_Packages_SMD:SOT-23-6
- removed SW3: RE-UPDIFY, Buttons_Switches_SMD:SW_SPST_EVPBF
- removed VTG1: GREEN, LEDs:LED_0805
- added D1: PMEG4005CEJX, Diodes_SMD:D_SOD-323F, F.Cu at (178.7, 74.6)
- added D3: ORANGE, WP934AD:WP934AD, F.Cu at (196.8, 76.8)
- added J1: ATMEL ICE, SAMTEC_SHF-105-01-L-D-RA:SAMTEC_SHF-105-01-L-D-RA, F.Cu at (149.2, 79.4)
- added J2: HVUPDI-OUT, SL_3_RA:SL_3_RA, F.Cu at (196.8, 85.1)
- added R1: 10K, Resistors_SMD:R_0603, F.Cu at (167.3, 94.0)
- added R2: 10K, Resistors_SMD:R_0603, F.Cu at (170.8, 90.3)
- added R7: 10K, Resistors_SMD:R_0603, F.Cu at (174.4, 90.2)
- added U4: ISL43210IHZ-T, TO_SOT_Packages_SMD:SOT-23-6, F.Cu at (159.2, 92.0)
- added U5: SN74LVC1G3157DBVR, TO_SOT_Packages_SMD:SOT-23-6, F.Cu at (171.2, 80.6)
- C4: value 68pF -> 0.1µF
- C6: value 4.7µF -> 68pF
- C7: value 0.1µF -> 4.7µF
- D2: value PMEG4005CEJX -> GREEN; footprint Diodes_SMD:D_SOD-323F -> WP934AD:WP934AD
- FID1, FID2, FID3, FID4: footprint Fiducial:Fiducial_1mm_Mask2mm -> Fiducials:Fiducial_1mm_Dia_2mm_Outer
- R3: value 10K -> 102K 1%
- R4: value 10K -> 11K 1%
- R5: value 102K 1% -> 1K
- R6: value 11K 1% -> 1K
- R8, R9: value 1K -> 180Ω
- SW1: value SN74LVC1G3157DBVR -> RE-UPDIFY; footprint TO_SOT_Packages_SMD:SOT-23-6 -> Buttons_Switches_ThroughHole:SW_Tactile_SPST_Angled_PTS645Vx58-2LFS
- moved FID2 150.3 mm to (179.2, 77.9)
- moved D2 144.4 mm to (196.8, 93.3)
- moved FID4 136.9 mm to (175.4, 84.3)
- moved FID1 125.0 mm to (167.3, 90.9)
- moved FID3 118.9 mm to (171.6, 87.2)
- moved C4 115.8 mm to (175.5, 81.3)
- moved U3 115.4 mm to (174.2, 75.5)
- moved U2 113.1 mm to (163.6, 86.8)
- moved C2 112.3 mm to (167.9, 87.9)
- moved C5 111.7 mm to (175.5, 79.0)
- moved C3 109.6 mm to (163.6, 92.7)
- moved F1 106.6 mm to (171.6, 84.2)
- moved C8 105.6 mm to (167.9, 85.5)
- moved C6 105.1 mm to (163.6, 90.3)
- moved C7 104.5 mm to (158.7, 95.5)
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Connections:
- C4 pad 1: /12V -> VTG
- C4 pad 2: Net-(C4-Pad2) -> GND
- C6 pad 2: GND -> Net-(C6-Pad2)
- C8 pad 1: VTG -> /12V
- D2 pad 1: /12V -> GND
- L1 pad 2: Net-(D2-Pad2) -> Net-(D1-Pad2)
- R3 pad 1: /UPDI-SENSE -> /12V
- R3 pad 2: /UPDI-HOST -> Net-(C6-Pad2)
- R4 pad 1: /PWR-SW-EN -> Net-(C6-Pad2)
- R5 pad 1: /12V -> VTG-PC
- R5 pad 2: Net-(C4-Pad2) -> GND
- R6 pad 1: Net-(C4-Pad2) -> VTG-PC
- R6 pad 2: GND -> Net-(D2-Pad2)
- R8 pad 1: VTG-PC -> Net-(R8-Pad1)
- R8 pad 2: GND -> Net-(R8-Pad2)
- R9 pad 1: VTG-PC -> Net-(D3-Pad2)
- R9 pad 2: Net-(R9-Pad2) -> /UPDI-EN
- SW1 pad 1: /UPDI-KEY -> GND
- SW1 pad 2: GND -> /UPDI-SENSE
- U2 pad 2: Net-(C4-Pad2) -> Net-(C6-Pad2)
- U2 pad 5: Net-(D2-Pad2) -> Net-(D1-Pad2)

Commit message: Layout WIP
Parts:
- removed FID4: Fiducial, Fiducials:Fiducial_1mm_Dia_2mm_Outer
- C1, C2, C3, C4, C5, C6, C7, C8: footprint Capacitors_SMD:C_0603 -> Capacitor_SMD:C_0603_1608Metric
- D1: footprint Diodes_SMD:D_SOD-323F -> Diode_SMD:D_SOD-323F
- F1, R1, R2, R3, R4, R5, R6, R7, R8, R9: footprint Resistors_SMD:R_0603 -> Resistor_SMD:R_0603_1608Metric
- FID1, FID2, FID3: footprint Fiducials:Fiducial_1mm_Dia_2mm_Outer -> Fiducial:Fiducial_1mm_Mask2mm
- J1: footprint SAMTEC_SHF-105-01-L-D-RA:SAMTEC_SHF-105-01-L-D-RA -> SAMTEC_SHF-105-01-X-D-TH:SAMTEC_SHF-105-01-X-D-TH
- L1: footprint L_1008_2520Metric:L_1008_2520Metric -> Inductor_SMD:L_1008_2520Metric
- SW1: footprint Buttons_Switches_ThroughHole:SW_Tactile_SPST_Angled_PTS645Vx58-2LFS -> Button_Switch_SMD:SW_SPST_B3SL-1002P
- U1: footprint Housings_SOIC:SOIC-8_3.9x4.9mm_Pitch1.27mm -> Package_SO:SO-8_3.9x4.9mm_P1.27mm
- U2, U3: footprint TO_SOT_Packages_SMD:SOT-23-5 -> Package_TO_SOT_SMD:SOT-23-5
- U4, U5: footprint TO_SOT_Packages_SMD:SOT-23-6 -> Package_TO_SOT_SMD:SOT-23-6
- moved R5 45.6 mm to (167.0, 50.2), turned to 180 degrees
- moved FID1 45.1 mm to (148.0, 50.2)
- moved R1 44.4 mm to (174.6, 50.2)
- moved SW1 44.4 mm to (160.7, 53.0)
- moved D2 43.2 mm to (189.2, 50.8)
- moved C3 40.1 mm to (167.0, 52.7), turned to 180 degrees
- moved FID3 37.1 mm to (179.1, 50.8)
- moved R6 36.7 mm to (182.2, 50.8), turned to 270 degrees
- moved C7 33.4 mm to (162.6, 62.2)
- moved R4 32.9 mm to (158.8, 62.2)
- moved R2 32.7 mm to (167.0, 57.8)
- moved C5 29.2 mm to (170.8, 50.2)
- moved R3 27.9 mm to (158.8, 64.8), turned to 180 degrees
- moved F1 27.4 mm to (149.7, 67.6)
- moved C4 27.4 mm to (167.0, 55.2), turned to 180 degrees
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Connections:
- J1 pad 10: Net-(J1-Pad10) -> GND
Other:
- board outline added: 43.2 x 22.9 mm

Commit message: Layout WIP
Parts:
- moved F1 17.0 mm to (152.4, 50.8), turned to 180 degrees
- moved R8 1.27 mm to (176.5, 68.6)
- moved C2 0.90 mm to (149.9, 68.6), turned to 90 degrees
- moved C8 0.64 mm to (165.7, 68.6)
- moved U4 0.64 mm to (172.1, 68.6)
- moved U2 0.51 mm to (154.3, 68.6)
- moved D1 0.38 mm to (162.6, 68.6)
Routing:
- net GND: track 0.00 -> 157.7 mm, vias 0 -> 15
- net VF: track 0.00 -> 64.7 mm, vias 0 -> 2
- net VTG: track 0.00 -> 38.1 mm, vias 0 -> 2
- net VTG-PC: track 0.00 -> 32.1 mm
- net /UPDI-EN: track 0.00 -> 24.3 mm, vias 0 -> 2
- net Net-(C6-Pad2): track 0.00 -> 24.1 mm, vias 0 -> 2
- net /12V: track 0.00 -> 23.6 mm
- net /UPDI-HOST: track 0.00 -> 23.2 mm
- net /UPDI-SENSE: track 0.00 -> 21.2 mm, vias 0 -> 4
- net /PROG: track 0.00 -> 20.6 mm, vias 0 -> 2
- net /PWR-SW-EN: track 0.00 -> 19.8 mm, vias 0 -> 2
- net Net-(R8-Pad2): track 0.00 -> 18.7 mm, vias 0 -> 2
- net /HVUPDI-TARGET: track 0.00 -> 13.2 mm
- net Net-(D1-Pad2): track 0.00 -> 8.11 mm
- net /HV-EN: track 0.00 -> 6.90 mm
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- added copper zone on B.Cu, net GND
- added copper zone on F.Cu, net GND
Other:
- net class Default: trace_width 0.2032 -> 0.25

Commit message: Layout WIP
Parts:
- D2: value GREEN -> TARGET PWR
- D3: value ORANGE -> UPDI EN
- J2: value HVUPDI-OUT -> TARGET
- SW1: value RE-UPDIFY -> RE-SEND
- U1: footprint Package_SO:SO-8_3.9x4.9mm_P1.27mm -> Package_SO:SOIC-8_3.9x4.9mm_P1.27mm
- moved SW1 0.38 mm to (160.7, 53.3)
- moved U3 0.25 mm to (170.8, 53.6)
- moved U1 0.13 mm to (169.0, 63.5)
Routing:
- net VTG: track 38.1 -> 40.4 mm
- net /UPDI-SENSE: track 21.2 -> 22.2 mm
- net Net-(C6-Pad2): track 24.1 -> 25.0 mm
- net VTG-PC: track 32.1 -> 31.4 mm
- net /PWR-SW-EN: track 19.8 -> 20.5 mm
- net /UPDI-EN: track 24.3 -> 24.9 mm
Other:
- board text added: "Updi-Key"

Commit message: Layout WIP
Routing:
- net GND: track 157.7 -> 237.0 mm, vias 15 -> 27
Other:
- board text added: "VTG GND UPDI"

Commit message: DRC
Other:
- net class Default: clearance 0.2032 -> 0.1524
- net class PWR16: clearance 0.2032 -> 0.1524
- net class PWR20: clearance 0.2032 -> 0.1524
- net class PWR24: clearance 0.2032 -> 0.1524
- net class PWR28: clearance 0.2032 -> 0.1524
- net class PWR32: clearance 0.2032 -> 0.1524
- rule trace_clearance: 0.2032 -> 0.1524

Commit message: Post build fixes
Parts:
- removed the C4 at (167.0, 55.2)
- removed the C5 at (170.8, 50.2)
- removed the R1 at (174.6, 50.2)
- removed the R5 at (167.0, 50.2)
- removed the U3 at (170.8, 53.6)
- added JP1: JP1, Connector_PinHeader_2.00mm:PinHeader_1x02_P2.00mm_Vertical, F.Cu at (170.1, 52.3)
- moved C3 2.41 mm to (167.0, 55.1)
- renumbered C6 to C4, C7 to C5, C8 to C6, D2 to D1, D1 to D2, R6 to R1, R7 to R5, R8 to R6, R9 to R7, U4 to U3, U5 to U4
Connections:
- net /HV-EN renamed /HV_EN
- net /HVUPDI-TARGET renamed /HVUPDI_TARGET
- net /UPDI-EN renamed /UPDI_EN
- net /UPDI-HOST renamed /UPDI_HOST
- net /UPDI-KEY renamed /UPDI_DAT
- net /UPDI-SENSE renamed /UPDI_SENSE
- net VF renamed /VF
- C3 pad 1: VTG -> /VTG
- F1 pad 2: VTG -> /VTG
- J1 pad 4: VTG -> /VTG
- J1 pad 7: /PROG -> Net-(J1-Pad7)
- J2 pad 3: VTG-PC -> /VTG
- R1 pad 1: VTG-PC -> /VTG
- U1 pad 2: /PWR-SW-EN -> Net-(U1-Pad2)
Routing:
- net /VTG: track 0.00 -> 64.7 mm, vias 0 -> 2
- net VTG: track 40.3 -> 0.00 mm, vias 2 -> 0
- net GND: track 237.0 -> 198.6 mm, vias 27 -> 20
- net VTG-PC: track 31.4 -> 0.00 mm
- net /PWR-SW-EN: track 20.5 -> 0.00 mm, vias 2 -> 0
- net /PROG: track 20.7 -> 13.5 mm, vias 2 -> 1
- net /UPDI_HOST: track 22.7 -> 27.0 mm
- net /VF: track 64.6 -> 66.2 mm
Other:
- board text added: "SELF PROGRAM"
