File: KiCad/Updifier/Updifier.sch (KiCad schematic (older format))
At the start: 36 parts, among them J2 UPDI-IN, J3 UPDI_IN6, J4 HVUPDI_OUT6, J5 HVUPDI-OUT, SW1 SN74LVC1G3157DBVR, SW2 ISL43210IHZ-T, SW3 PTS810SJG250SMTRLFS, U1 ATtiny202-SS, U2 NCP1406SNT1G, U3 MIC2091-1YM5-TR

Commit message: WIP
Parts:
- removed J2: UPDI-IN, Connector_PinHeader_2.54mm:PinHeader_1x03_P2.54mm_Horizontal, symbol Connector_Generic:Conn_01x03
- removed J4: HVUPDI_OUT6, Connector_PinHeader_2.54mm:PinHeader_2x03_P2.54mm_Vertical, symbol Connector_Generic:Conn_02x03_Odd_Even
- removed SW3: PTS810SJG250SMTRLFS, 0_mouser:PTS810SJG250SMTRLFS, symbol SamacSys_Parts:PTS810SJG250SMTRLFS
- added SW3: RE-UPDIFY, Buttons_Switches_SMD:SW_SPST_EVPBF, symbol Switch:SW_SPST
- C1, C2, C3, C4, C5, C6, C7, C8: footprint Capacitor_SMD:C_0603_1608Metric -> Capacitors_SMD:C_0603
- D2: footprint Diode_SMD:D_SOD-323F -> Diodes_SMD:D_SOD-323F
- F1: footprint Fuse:Fuse_0603_1608Metric -> Resistors_SMD:R_0603
- HV1, VTG1: footprint LED_SMD:LED_0603_1608Metric -> LEDs:LED_0805
- J3: footprint Connector_PinHeader_2.54mm:PinHeader_2x03_P2.54mm_Vertical -> Pin_Headers:Pin_Header_Angled_2x05_Pitch1.00mm
- J5: footprint Connector_PinSocket_2.54mm:PinSocket_1x03_P2.54mm_Horizontal -> 78208-103HLF:78208-103HLF
- L1: footprint Inductor_SMD:L_1008_2520Metric -> L_1008_2520Metric:L_1008_2520Metric
- R10, R11, R12, R3, R4, R5, R6, R8, R9: footprint Resistor_SMD:R_0603_1608Metric -> Resistors_SMD:R_0603
- SW1, SW2: footprint 0_mouser:SOT95P280X145-6N -> TO_SOT_Packages_SMD:SOT-23-6
- U1: footprint Package_SO:SOIC-8_3.9x4.9mm_P1.27mm -> Housings_SOIC:SOIC-8_3.9x4.9mm_Pitch1.27mm
- U2: footprint 0_mouser:SOT95P275X110-5N -> TO_SOT_Packages_SMD:SOT-23-5
- U3: footprint 0_mouser:SOT95P280X130-5N -> TO_SOT_Packages_SMD:SOT-23-5
Connections:
- wire segments 144 -> 125
- no-connect marks 5 -> 3
Other:
- moved on the sheet: J3

Commit message: WIP
Parts:
- removed J3: UPDI_IN6, Pin_Headers:Pin_Header_Angled_2x05_Pitch1.00mm, symbol Connector_Generic:Conn_02x03_Odd_Even
- added J1: ATMEL ICE, SAMTEC_SHF-105-01-L-D-RA:SAMTEC_SHF-105-01-L-D-RA, symbol Connector_Generic:Conn_02x05_Counter_Clockwise
- D2: renamed from VTG1; footprint LEDs:LED_0805 -> WP934AD:WP934AD
- D3: renamed from HV1; footprint LEDs:LED_0805 -> WP934AD:WP934AD
- FID1, FID2, FID3, FID4: footprint Fiducial:Fiducial_1mm_Mask2mm -> Fiducials:Fiducial_1mm_Dia_2mm_Outer
- J2: renamed from J5; footprint 78208-103HLF:78208-103HLF -> SL_3_RA:SL_3_RA
- SW1: renamed from SW3; footprint Buttons_Switches_SMD:SW_SPST_EVPBF -> Buttons_Switches_ThroughHole:SW_Tactile_SPST_Angled_PTS645Vx58-2LFS
- renumbered C8 to C4, C4 to C6, C6 to C7, C7 to C8, D2 to D1, R4 to R1, R3 to R2, R5 to R3, R6 to R4, R8 to R5, R9 to R6, R10 to R7, R12 to R8, R11 to R9, SW2 to U4, SW1 to U5
Connections:
- wire segments 125 -> 129
Other:
- note added: "CHECH MECH BEFORE FABRICATION"
- note added: "CHECK FOOTPRINT AGAINST\nCOMMONLY AVAILABLE PRODUCT"
- note added: "VERIFY ATMEL-ICE USES SAME PIN ODERING AS SAMTEC SPECIFICATION"

Commit message: Layout WIP
Parts:
- removed FID4: Fiducial, Fiducials:Fiducial_1mm_Dia_2mm_Outer, symbol Mechanical:Fiducial
- removed J1: ATMEL ICE, SAMTEC_SHF-105-01-L-D-RA:SAMTEC_SHF-105-01-L-D-RA, symbol Connector_Generic:Conn_02x05_Counter_Clockwise
- added J1: ATMEL ICE, SAMTEC_SHF-105-01-X-D-TH:SAMTEC_SHF-105-01-X-D-TH, symbol Connector_Generic:Conn_02x05_Odd_Even
- C1, C2, C3, C4, C5, C6, C7, C8: footprint Capacitors_SMD:C_0603 -> Capacitor_SMD:C_0603_1608Metric
- D1: footprint Diodes_SMD:D_SOD-323F -> Diode_SMD:D_SOD-323F
- F1, R1, R2, R3, R4, R5, R6, R7, R8, R9: footprint Resistors_SMD:R_0603 -> Resistor_SMD:R_0603_1608Metric
- FID1, FID2, FID3: footprint Fiducials:Fiducial_1mm_Dia_2mm_Outer -> Fiducial:Fiducial_1mm_Mask2mm
- L1: footprint L_1008_2520Metric:L_1008_2520Metric -> Inductor_SMD:L_1008_2520Metric
- SW1: footprint Buttons_Switches_ThroughHole:SW_Tactile_SPST_Angled_PTS645Vx58-2LFS -> Button_Switch_SMD:SW_SPST_B3SL-1002P
- U1: footprint Housings_SOIC:SOIC-8_3.9x4.9mm_Pitch1.27mm -> Package_SO:SO-8_3.9x4.9mm_P1.27mm
- U2, U3: footprint TO_SOT_Packages_SMD:SOT-23-5 -> Package_TO_SOT_SMD:SOT-23-5
- U4, U5: footprint TO_SOT_Packages_SMD:SOT-23-6 -> Package_TO_SOT_SMD:SOT-23-6
Connections:
- wire segments 129 -> 131
- no-connect marks 3 -> 1

Commit message: Layout WIP
Parts:
- D2: value GREEN -> TARGET PWR
- D3: value ORANGE -> UPDI EN
- J2: value HVUPDI-OUT -> TARGET
- SW1: value RE-UPDIFY -> RE-SEND
- U1: footprint Package_SO:SO-8_3.9x4.9mm_P1.27mm -> Package_SO:SOIC-8_3.9x4.9mm_P1.27mm
Changed lines of the file:
@@
 F 0 "U1" H 1850 3150 50  0000 R CNN
 F 1 "ATtiny202-SS" H 2850 3175 50  0000 R CNN
-F 2 "Package_SO:SO-8_3.9x4.9mm_P1.27mm" H 2250 2600 50  0001 C CIN
+F 2 "Package_SO:SOIC-8_3.9x4.9mm_P1.27mm" H 2250 2600 50  0001 C CIN
 F 3 "http://ww1.microchip.com/downloads/en/DeviceDoc/ATtiny202-402-AVR-MCU-with-Core-Independent-Peripherals_and-picoPower-40001969A.pdf" H 2250 2600 50  0001 C CNN
 F 4 "IC MCU 8BIT 2KB FLASH 8SOIC" H 2250 2600 50  0001 C CNN "Description"
@@
 P 6100 5650
 F 0 "D2" V 6150 5550 50  0000 C CNN
-F 1 "GREEN" V 5925 5425 50  0000 C CNN
+F 1 "TARGET PWR" V 5925 5425 50  0000 C CNN
 F 2 "WP934AD:WP934AD" H 6100 5650 50  0001 C CNN
 F 3 "https://dammedia.osram.info/media/resource/hires/osram-dam-2493948/LG%20Q396.pdf" H 6100 5650 50  0001 C CNN
@@
 P 9300 2000
 F 0 "J2" H 9450 2000 50  0000 C CNN
-F 1 "HVUPDI-OUT" H 9450 2200 50  0000 C CNN
+F 1 "TARGET" H 9450 2200 50  0000 C CNN
 F 2 "SL_3_RA:SL_3_RA" H 9300 2000 50  0001 C CNN
 F 3 "~" H 9300 2000 50  0001 C CNN
@@
 P 9050 2800
 F 0 "D3" H 9050 2700 50  0000 C CNN
-F 1 "ORANGE" H 9043 2925 50  0000 C CNN
+F 1 "UPDI EN" H 9043 2925 50  0000 C CNN
 F 2 "WP934AD:WP934AD" H 9050 2800 50  0001 C CNN
 F 3 "http://www.kingbrightusa.com/images/catalog/SPEC/APTD1608SECK-J4-PF.pdf" H 9050 2800 50  0001 C CNN
@@
 P 3750 4100
 F 0 "SW1" V 3796 4012 50  0000 R CNN
-F 1 "RE-UPDIFY" V 3705 4012 50  0000 R CNN
+F 1 "RE-SEND" V 3705 4012 50  0000 R CNN
 F 2 "Button_Switch_SMD:SW_SPST_B3SL-1002P" H 3750 4100 50  0001 C CNN
 F 3 "~" H 3750 4100 50  0001 C CNN

Commit message: Layout WIP
Other:
- note removed: "CHECH MECH BEFORE FABRICATION"
- note removed: "CHECK FOOTPRINT AGAINST\nCOMMONLY AVAILABLE PRODUCT"
- note removed: "RE-UPDIFY"
- note removed: "VERIFY ATMEL-ICE USES SAME PIN ODERING AS SAMTEC SPECIFICATION"
Changed lines of the file:
@@
 Wire Wire Line
 	8000 1900 9100 1900
-Text Notes 3175 4100 0    50   ~ 0
-RE-UPDIFY
 NoConn ~ 5550 5100
 $Comp
@@
 Wire Wire Line
 	2850 2700 3425 2700
-Text Notes 9875 4725 2    50   ~ 0
-VERIFY ATMEL-ICE USES SAME PIN ODERING AS SAMTEC SPECIFICATION
-Text Notes 9850 2650 1    50   ~ 0
-CHECH MECH BEFORE FABRICATION
-Text Notes 3650 4300 2    50   ~ 0
-CHECK FOOTPRINT AGAINST\nCOMMONLY AVAILABLE PRODUCT
 $Comp
 L Connector_Generic:Conn_02x05_Odd_Even J1

Commit message: Post build fixes
Parts:
- removed C4: 0.1µF, Capacitor_SMD:C_0603_1608Metric, symbol Device:C_Small
- removed C5: 10µF, Capacitor_SMD:C_0603_1608Metric, symbol Device:C_Small
- removed R1: 10K, Resistor_SMD:R_0603_1608Metric, symbol Device:R_Small_US
- removed R5: 1K, Resistor_SMD:R_0603_1608Metric, symbol Device:R_Small_US
- removed U3: MIC2091-1YM5-TR, Package_TO_SOT_SMD:SOT-23-5, symbol SamacSys_Parts:MIC2091-1YM5-TR
- added JP1: JP1, Connector_PinHeader_2.00mm:PinHeader_1x02_P2.00mm_Vertical, symbol Device:Jumper
- renumbered C6 to C4, C7 to C5, C8 to C6, D2 to D1, D1 to D2, R6 to R1, R7 to R5, R8 to R6, R9 to R7, U4 to U3, U5 to U4
Connections:
- net labels added: HVUPDI_TARGET, HV_EN, UPDI_DAT, UPDI_EN, UPDI_HOST, UPDI_SENSE
- net labels removed: HV-EN, HVUPDI-TARGET, PWR-SW-EN, UPDI-EN, UPDI-HOST, UPDI-KEY, UPDI-SENSE, VTG-PC
- wire segments 131 -> 106
- no-connect marks 1 -> 0
Other:
- moved on the sheet: C1, C2, C3, C4, C5, C6, D1, D2, D3, F1, J2, L1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

Commit message: Release
Parts:
- R1: value 1K -> 220
Changed lines of the file:
@@
 P 1650 4300
 F 0 "R1" H 1700 4400 50  0000 L CNN
-F 1 "1K" H 1650 4200 50  0000 L CNN
+F 1 "220" H 1650 4200 50  0000 L CNN
 F 2 "Resistor_SMD:R_0603_1608Metric" H 1650 4300 50  0001 C CNN
 F 3 "http://www.koaspeer.com/pdfs/RK73B.pdf" H 1650 4300 50  0001 C CNN
